Commit message: feat: add base_rotation_link to URDF and introduce RViz visualization launch configuration

File: devotics_arm_description/urdf/devotics_arm_v1.urdf.xacro (robot description, xacro)
@@ -78,3 +78,31 @@
     <dynamics damping="0.1" friction="0.1" />
   </joint>
+    <!-- ========================================== -->
+  <!-- Base Rotation Link (Turret)                -->
+  <!-- ========================================== -->
+  <link name="base_rotation_link">
+    <!-- Turret turntable disk -->
+    <visual>
+      <origin xyz="0 0 0.006" rpy="0 0 0" />
+      <geometry>
+        <cylinder radius="0.050" length="0.012" />
+      </geometry>
+      <material name="devotics_orange" />
+    </visual>
+    <!-- Shoulder support columns (80mm rise to J2 pivot) -->
+    <visual>
+      <origin xyz="0 0 0.046" rpy="0 0 0" />
+      <geometry>
+        <box size="0.045 0.075 0.068" />
+      </geometry>
+      <material name="dark_gray" />
+    </visual>
+    <collision>
+      <origin xyz="0 0 0.040" rpy="0 0 0" />
+      <geometry>
+        <box size="0.060 0.080 0.080" />
+      </geometry>
+    </collision>
+    <xacro:box_inertia m="0.28" x="0.060" y="0.080" z="0.080" />
+  </link>
 </robot>

Commit message: feat: add links, joints, and gripper assembly for joints 2 through 5 in arm URDF

File: devotics_arm_description/urdf/devotics_arm_v1.urdf.xacro (robot description, xacro)
@@ -106,3 +106,252 @@
     <xacro:box_inertia m="0.28" x="0.060" y="0.080" z="0.080" />
   </link>
+    <!-- ========================================== -->
+  <!-- Joint 2: Shoulder Pitch (MG996R + Springs) -->
+  <!-- ========================================== -->
+  <joint name="joint_2" type="revolute">
+    <parent link="base_rotation_link" />
+    <child link="upper_arm_link" />
+    <origin xyz="0 0 ${J1_TO_J2_Z}" rpy="0 0 0" />
+    <axis xyz="0 1 0" />
+    <limit lower="-1.5708" upper="1.5708" effort="3.0" velocity="3.14" />
+    <dynamics damping="0.15" friction="0.1" />
+  </joint>
+  <!-- ========================================== -->
+  <!-- Upper Arm Link (185 mm Pivot-to-Pivot)     -->
+  <!-- ========================================== -->
+  <link name="upper_arm_link">
+    <!-- Shoulder pivot boss -->
+    <visual>
+      <origin xyz="0 0 0" rpy="1.5708 0 0" />
+      <geometry>
+        <cylinder radius="0.025" length="0.050" />
+      </geometry>
+      <material name="metallic_silver" />
+    </visual>
+    <!-- Main upper arm bone (185mm center span) -->
+    <visual>
+      <origin xyz="0 0 ${J2_TO_J3_LEN / 2.0}" rpy="0 0 0" />
+      <geometry>
+        <box size="0.035 0.050 ${J2_TO_J3_LEN}" />
+      </geometry>
+      <material name="devotics_orange" />
+    </visual>
+    <!-- Elbow pivot boss -->
+    <visual>
+      <origin xyz="0 0 ${J2_TO_J3_LEN}" rpy="1.5708 0 0" />
+      <geometry>
+        <cylinder radius="0.025" length="0.050" />
+      </geometry>
+      <material name="metallic_silver" />
+    </visual>
+    <collision>
+      <origin xyz="0 0 ${J2_TO_J3_LEN / 2.0}" rpy="0 0 0" />
+      <geometry>
+        <box size="0.050 0.060 ${J2_TO_J3_LEN + 0.050}" />
+      </geometry>
+    </collision>
+    <xacro:box_inertia m="0.25" x="0.050" y="0.060" z="${J2_TO_J3_LEN + 0.050}" />
+  </link>
+    <!-- ========================================== -->
+  <!-- Joint 3: Elbow Pitch (MG996R)              -->
+  <!-- ========================================== -->
+  <joint name="joint_3" type="revolute">
+    <parent link="upper_arm_link" />
+    <child link="forearm_link" />
+    <origin xyz="0 0 ${J2_TO_J3_LEN}" rpy="0 0 0" />
+    <axis xyz="0 1 0" />
+    <limit lower="-2.0944" upper="2.0944" effort="2.5" velocity="3.14" />
+    <dynamics damping="0.1" friction="0.1" />
+  </joint>
+  <!-- ========================================== -->
+  <!-- Forearm Link (138 mm Pivot-to-Pivot)       -->
+  <!-- ========================================== -->
+  <link name="forearm_link">
+    <!-- Elbow hinge boss -->
+    <visual>
+      <origin xyz="0 0 0" rpy="1.5708 0 0" />
+      <geometry>
+        <cylinder radius="0.022" length="0.045" />
+      </geometry>
+      <material name="metallic_silver" />
+    </visual>
+    <!-- Main forearm body (138mm span) -->
+    <visual>
+      <origin xyz="0 0 ${J3_TO_J4_LEN / 2.0}" rpy="0 0 0" />
+      <geometry>
+        <box size="0.030 0.045 ${J3_TO_J4_LEN}" />
+      </geometry>
+      <material name="dark_gray" />
+    </visual>
+    <!-- Wrist hinge boss -->
+    <visual>
+      <origin xyz="0 0 ${J3_TO_J4_LEN}" rpy="1.5708 0 0" />
+      <geometry>
+        <cylinder radius="0.020" length="0.045" />
+      </geometry>
+      <material name="metallic_silver" />
+    </visual>
+    <collision>
+      <origin xyz="0 0 ${J3_TO_J4_LEN / 2.0}" rpy="0 0 0" />
+      <geometry>
+        <box size="0.045 0.055 ${J3_TO_J4_LEN + 0.040}" />
+      </geometry>
+    </collision>
+    <xacro:box_inertia m="0.20" x="0.045" y="0.055" z="${J3_TO_J4_LEN + 0.040}" />
+  </link>
+  <!-- ========================================== -->
+  <!-- Joint 4: Wrist Pitch (MG996R)              -->
+  <!-- ========================================== -->
+  <joint name="joint_4" type="revolute">
+    <parent link="forearm_link" />
+    <child link="wrist_pitch_link" />
+    <origin xyz="0 0 ${J3_TO_J4_LEN}" rpy="0 0 0" />
+    <axis xyz="0 1 0" />
+    <limit lower="-1.5708" upper="1.5708" effort="2.0" velocity="3.14" />
+    <dynamics damping="0.08" friction="0.08" />
+  </joint>
+  <!-- ========================================== -->
+  <!-- Wrist Pitch Link (65 mm offset to roll)    -->
+  <!-- ========================================== -->
+  <link name="wrist_pitch_link">
+    <!-- Pitch hinge boss -->
+    <visual>
+      <origin xyz="0 0 0" rpy="1.5708 0 0" />
+      <geometry>
+        <cylinder radius="0.018" length="0.040" />
+      </geometry>
+      <material name="devotics_orange" />
+    </visual>
+    <!-- Housing body projecting forward along X -->
+    <visual>
+      <origin xyz="${J4_TO_J5_OFFSET / 2.0} 0 0" rpy="0 0 0" />
+      <geometry>
+        <box size="${J4_TO_J5_OFFSET} 0.042 0.045" />
+      </geometry>
+      <material name="devotics_orange" />
+    </visual>
+    <collision>
+      <origin xyz="${J4_TO_J5_OFFSET / 2.0} 0 0" rpy="0 0 0" />
+      <geometry>
+        <box size="${J4_TO_J5_OFFSET} 0.045 0.045" />
+      </geometry>
+    </collision>
+    <xacro:box_inertia m="0.12" x="${J4_TO_J5_OFFSET}" y="0.045" z="0.045" />
+  </link>
+  <!-- ========================================== -->
+  <!-- Joint 5: Wrist Roll (MG996R)               -->
+  <!-- ========================================== -->
+  <joint name="joint_5" type="revolute">
+    <parent link="wrist_pitch_link" />
+    <child link="wrist_roll_link" />
+    <origin xyz="${J4_TO_J5_OFFSET} 0 0" rpy="0 0 0" />
+    <axis xyz="1 0 0" />
+    <limit lower="-3.14159" upper="3.14159" effort="1.5" velocity="3.14" />
+    <dynamics damping="0.05" friction="0.05" />
+  </joint>
+  <!-- ========================================== -->
+  <!-- Wrist Roll Link (Flange)                   -->
+  <!-- ========================================== -->
+  <link name="wrist_roll_link">
+    <visual>
+      <origin xyz="${J5_TO_GRIPPER_BASE / 2.0} 0 0" rpy="0 1.5708 0" />
+      <geometry>
+        <cylinder radius="0.018" length="${J5_TO_GRIPPER_BASE}" />
+      </geometry>
+      <material name="metallic_silver" />
+    </visual>
+    <collision>
+      <origin xyz="${J5_TO_GRIPPER_BASE / 2.0} 0 0" rpy="0 1.5708 0" />
+      <geometry>
+        <cylinder radius="0.020" length="${J5_TO_GRIPPER_BASE}" />
+      </geometry>
+    </collision>
+    <xacro:cylinder_inertia m="0.04" r="0.020" h="${J5_TO_GRIPPER_BASE}" />
+  </link>
+    <!-- ========================================== -->
+  <!-- Fixed Flange Joint to Gripper Base         -->
+  <!-- ========================================== -->
+  <joint name="joint_gripper_base" type="fixed">
+    <parent link="wrist_roll_link" />
+    <child link="gripper_base_link" />
+    <origin xyz="${J5_TO_GRIPPER_BASE} 0 0" rpy="0 0 0" />
+  </joint>
+  <!-- ========================================== -->
+  <!-- Gripper Base Body (MG90S housing)          -->
+  <!-- ========================================== -->
+  <link name="gripper_base_link">
+    <visual>
+      <origin xyz="0.020 0 0" rpy="0 0 0" />
+      <geometry>
+        <box size="0.040 0.045 0.035" />
+      </geometry>
+      <material name="dark_gray" />
+    </visual>
+    <collision>
+      <origin xyz="0.020 0 0" rpy="0 0 0" />
+      <geometry>
+        <box size="0.040 0.045 0.035" />
+      </geometry>
+    </collision>
+    <xacro:box_inertia m="0.06" x="0.040" y="0.045" z="0.035" />
+  </link>
+  <!-- ========================================== -->
+  <!-- Actuated Gripper Jaws (Left + Right Mimic) -->
+  <!-- ========================================== -->
+  <joint name="gripper_left_finger_joint" type="prismatic">
+    <parent link="gripper_base_link" />
+    <child link="gripper_left_finger_link" />
+    <origin xyz="0.040 0.015 0" rpy="0 0 0" />
+    <axis xyz="0 1 0" />
+    <limit lower="0.0" upper="0.025" effort="1.0" velocity="0.1" />
+  </joint>
+  <link name="gripper_left_finger_link">
+    <visual>
+      <origin xyz="0.020 0 0" rpy="0 0 0" />
+      <geometry>
+        <box size="0.040 0.006 0.015" />
+      </geometry>
+      <material name="light_gray" />
+    </visual>
+    <collision>
+      <origin xyz="0.020 0 0" rpy="0 0 0" />
+      <geometry>
+        <box size="0.040 0.006 0.015" />
+      </geometry>
+    </collision>
+    <xacro:box_inertia m="0.01" x="0.040" y="0.006" z="0.015" />
+  </link>
+  <joint name="gripper_right_finger_joint" type="prismatic">
+    <parent link="gripper_base_link" />
+    <child link="gripper_right_finger_link" />
+    <origin xyz="0.040 -0.015 0" rpy="0 0 0" />
+    <axis xyz="0 -1 0" />
+    <limit lower="0.0" upper="0.025" effort="1.0" velocity="0.1" />
+    <mimic joint="gripper_left_finger_joint" multiplier="1.0" offset="0.0" />
+  </joint>
+  <link name="gripper_right_finger_link">
+    <visual>
+      <origin xyz="0.020 0 0" rpy="0 0 0" />
+      <geometry>
+        <box size="0.040 0.006 0.015" />
+      </geometry>
+      <material name="light_gray" />
+    </visual>
+    <collision>
+      <origin xyz="0.020 0 0" rpy="0 0 0" />
+      <geometry>
+        <box size="0.040 0.006 0.015" />
+      </geometry>
+    </collision>
+    <xacro:box_inertia m="0.01" x="0.040" y="0.006" z="0.015" />
+  </link>
+  <!-- ========================================== -->
+  <!-- TCP / Tool0 Frame (Grasp Contact Center)   -->
+  <!-- ========================================== -->
+  <joint name="tcp_joint" type="fixed">
+    <parent link="gripper_base_link" />
+    <child tool="tool" link="tool0" />
+    <origin xyz="${GRIPPER_BASE_TO_TCP} 0 0" rpy="0 0 0" />
+  </joint>
+  <link name="tool0" />
 </robot>

Commit message: feat: add visual meshes and update URDF and visualization configuration

File: devotics_arm_description/urdf/devotics_arm_v1.urdf.xacro (robot description, xacro)
@@ -39,21 +39,21 @@
     <origin xyz="0 0 0" rpy="0 0 0" />
   </joint>
-  <!-- ========================================== -->
+    <!-- ========================================== -->
   <!-- Base Link (Stationary Baseplate + Housing) -->
   <!-- ========================================== -->
   <link name="base_link">
-    <!-- Base mounting plate (150x150x12 mm) -->
-    <visual>
-      <origin xyz="0 0 0.006" rpy="0 0 0" />
-      <geometry>
-        <box size="0.150 0.150 0.012" />
+    <!-- Visual 1: Base Mount Plate (Base_02.stl) -->
+    <visual>
+      <origin xyz="0 0 0" rpy="1.5708 0 0" />
+      <geometry>
+        <mesh filename="package://devotics_arm_description/meshes/visual/Base_02.stl" scale="0.001 0.001 0.001" />
       </geometry>
       <material name="dark_gray" />
     </visual>
-    <!-- Bearing & J1 housing (120mm diam, 43mm rise) -->
-    <visual>
-      <origin xyz="0 0 0.0335" rpy="0 0 0" />
-      <geometry>
-        <cylinder radius="0.060" length="0.043" />
+    <!-- Visual 2: Base Bearing Housing (Base_01.stl) -->
+    <visual>
+      <origin xyz="0 0 0" rpy="1.5708 0 0" />
+      <geometry>
+        <mesh filename="package://devotics_arm_description/meshes/visual/Base_01.stl" scale="0.001 0.001 0.001" />
       </geometry>
       <material name="light_gray" />
@@ -78,23 +78,15 @@
     <dynamics damping="0.1" friction="0.1" />
   </joint>
-    <!-- ========================================== -->
+   <!-- ========================================== -->
   <!-- Base Rotation Link (Turret)                -->
   <!-- ========================================== -->
   <link name="base_rotation_link">
-    <!-- Turret turntable disk -->
-    <visual>
-      <origin xyz="0 0 0.006" rpy="0 0 0" />
-      <geometry>
-        <cylinder radius="0.050" length="0.012" />
+    <!-- Turret Chassis (Base_03.stl) -->
+    <visual>
+      <origin xyz="0 0 0" rpy="1.5708 0 1.5708" />
+      <geometry>
+        <mesh filename="package://devotics_arm_description/meshes/visual/Base_03.stl" scale="0.001 0.001 0.001" />
       </geometry>
       <material name="devotics_orange" />
-    </visual>
-    <!-- Shoulder support columns (80mm rise to J2 pivot) -->
-    <visual>
-      <origin xyz="0 0 0.046" rpy="0 0 0" />
-      <geometry>
-        <box size="0.045 0.075 0.068" />
-      </geometry>
-      <material name="dark_gray" />
     </visual>
     <collision>
@@ -117,31 +109,14 @@
     <dynamics damping="0.15" friction="0.1" />
   </joint>
-  <!-- ========================================== -->
+   <!-- ========================================== -->
   <!-- Upper Arm Link (185 mm Pivot-to-Pivot)     -->
   <!-- ========================================== -->
   <link name="upper_arm_link">
-    <!-- Shoulder pivot boss -->
-    <visual>
-      <origin xyz="0 0 0" rpy="1.5708 0 0" />
-      <geometry>
-        <cylinder radius="0.025" length="0.050" />
-      </geometry>
-      <material name="metallic_silver" />
-    </visual>
-    <!-- Main upper arm bone (185mm center span) -->
-    <visual>
-      <origin xyz="0 0 ${J2_TO_J3_LEN / 2.0}" rpy="0 0 0" />
-      <geometry>
-        <box size="0.035 0.050 ${J2_TO_J3_LEN}" />
-      </geometry>
-      <material name="devotics_orange" />
-    </visual>
-    <!-- Elbow pivot boss -->
-    <visual>
-      <origin xyz="0 0 ${J2_TO_J3_LEN}" rpy="1.5708 0 0" />
-      <geometry>
-        <cylinder radius="0.025" length="0.050" />
-      </geometry>
-      <material name="metallic_silver" />
+    <visual>
+      <origin xyz="0 0 0" rpy="1.5708 0 0" />
+      <geometry>
+        <mesh filename="package://devotics_arm_description/meshes/visual/Brazo_01.stl" scale="0.001 0.001 0.001" />
+      </geometry>
+      <material name="light_gray" />
     </visual>
     <collision>

Commit message: refactor: update robot base dimensions in URDF, adjust RViz view settings, and add launch script

File: devotics_arm_description/urdf/devotics_arm_v1.urdf.xacro (robot description, xacro)
@@ -4,5 +4,5 @@
   <xacro:include filename="materials.xacro" />
   <!-- 2. Kinematic Constants (Meters) — From Stage 1 Reverse Engineering -->
-  <xacro:property name="BASE_TO_J1_Z" value="0.055" />       <!-- 55.0 mm: Table to Yaw plane -->
+  <xacro:property name="BASE_TO_J1_Z" value="0.012" />       <!-- 55.0 mm: Table to Yaw plane -->
   <xacro:property name="J1_TO_J2_Z" value="0.080" />         <!-- 80.0 mm: Turret rise to Shoulder -->
   <xacro:property name="J2_TO_J3_LEN" value="0.185" />       <!-- 185.0 mm: Upper arm pivot-to-pivot -->
@@ -39,9 +39,9 @@
     <origin xyz="0 0 0" rpy="0 0 0" />
   </joint>
-    <!-- ========================================== -->
-  <!-- Base Link (Stationary Baseplate + Housing) -->
+  <!-- ========================================== -->
+  <!-- Base Link (Stationary Table Mount Flange)  -->
   <!-- ========================================== -->
   <link name="base_link">
-    <!-- Visual 1: Base Mount Plate (Base_02.stl) -->
+    <!-- Base Mount Plate (Base_02.stl) -->
     <visual>
       <origin xyz="0 0 0" rpy="1.5708 0 0" />
@@ -51,19 +51,11 @@
       <material name="dark_gray" />
     </visual>
-    <!-- Visual 2: Base Bearing Housing (Base_01.stl) -->
-    <visual>
-      <origin xyz="0 0 0" rpy="1.5708 0 0" />
-      <geometry>
-        <mesh filename="package://devotics_arm_description/meshes/visual/Base_01.stl" scale="0.001 0.001 0.001" />
-      </geometry>
-      <material name="light_gray" />
-    </visual>
-    <collision>
-      <origin xyz="0 0 0.0275" rpy="0 0 0" />
-      <geometry>
-        <cylinder radius="0.075" length="0.055" />
-      </geometry>
-    </collision>
-    <xacro:cylinder_inertia m="0.45" r="0.075" h="0.055" />
+    <collision>
+      <origin xyz="0 0 0.006" rpy="0 0 0" />
+      <geometry>
+        <cylinder radius="0.075" length="0.012" />
+      </geometry>
+    </collision>
+    <xacro:cylinder_inertia m="0.15" r="0.075" h="0.012" />
   </link>
   <!-- ========================================== -->
@@ -78,23 +70,39 @@
     <dynamics damping="0.1" friction="0.1" />
   </joint>
-   <!-- ========================================== -->
-  <!-- Base Rotation Link (Turret)                -->
+  <!-- ========================================== -->
+  <!-- Base Rotation Link (Drum + 2 Side Towers)  -->
   <!-- ========================================== -->
   <link name="base_rotation_link">
-    <!-- Turret Chassis (Base_03.stl) -->
+    <!-- Visual 1: Main Rotating Housing Drum (Base_01.stl) -->
     <visual>
       <origin xyz="0 0 0" rpy="1.5708 0 1.5708" />
       <geometry>
+        <mesh filename="package://devotics_arm_description/meshes/visual/Base_01.stl" scale="0.001 0.001 0.001" />
+      </geometry>
+      <material name="dark_gray" />
+    </visual>
+    <!-- Visual 2: Left Tower (aligned with Left shelf) -->
+    <visual>
+      <origin xyz="0 0.0525 0" rpy="1.5708 0 1.5708" />
+      <geometry>
         <mesh filename="package://devotics_arm_description/meshes/visual/Base_03.stl" scale="0.001 0.001 0.001" />
       </geometry>
       <material name="devotics_orange" />
     </visual>
+    <!-- Visual 3: Right Tower (aligned with Right shelf) -->
+    <visual>
+      <origin xyz="0 -0.0525 0" rpy="1.5708 0 -1.5708" />
+      <geometry>
+        <mesh filename="package://devotics_arm_description/meshes/visual/Base_03.stl" scale="0.001 0.001 0.001" />
+      </geometry>
+      <material name="devotics_orange" />
+    </visual>
     <collision>
       <origin xyz="0 0 0.040" rpy="0 0 0" />
       <geometry>
-        <box size="0.060 0.080 0.080" />
-      </geometry>
-    </collision>
-    <xacro:box_inertia m="0.28" x="0.060" y="0.080" z="0.080" />
+        <cylinder radius="0.060" length="0.080" />
+      </geometry>
+    </collision>
+    <xacro:cylinder_inertia m="0.45" r="0.060" h="0.080" />
   </link>
     <!-- ========================================== -->

Commit message: feat: add thrust bearing and servo horn retainer visual components to base link in URDF

File: devotics_arm_description/urdf/devotics_arm_v1.urdf.xacro (robot description, xacro)
@@ -5,4 +5,5 @@
   <!-- 2. Kinematic Constants (Meters) — From Stage 1 Reverse Engineering -->
   <xacro:property name="BASE_TO_J1_Z" value="0.012" />       <!-- 55.0 mm: Table to Yaw plane -->
+  <xacro:property name="BASE_TO_J1_Z" value="0.006" />       <!-- 6.0 mm: Ball bearing rolling plane -->
   <xacro:property name="J1_TO_J2_Z" value="0.080" />         <!-- 80.0 mm: Turret rise to Shoulder -->
   <xacro:property name="J2_TO_J3_LEN" value="0.185" />       <!-- 185.0 mm: Upper arm pivot-to-pivot -->
@@ -39,9 +40,9 @@
     <origin xyz="0 0 0" rpy="0 0 0" />
   </joint>
-  <!-- ========================================== -->
-  <!-- Base Link (Stationary Table Mount Flange)  -->
+    <!-- ========================================== -->
+  <!-- Base Link (Stationary Baseplate Assembly)  -->
   <!-- ========================================== -->
   <link name="base_link">
-    <!-- Base Mount Plate (Base_02.stl) -->
+    <!-- 1. Table Mount Baseplate (Base_02.stl) -->
     <visual>
       <origin xyz="0 0 0" rpy="1.5708 0 0" />
@@ -51,4 +52,20 @@
       <material name="dark_gray" />
     </visual>
+    <!-- 2. Thrust Ball Bearing Cage (Jaula_bolas.stl) seated in the raceway -->
+    <visual>
+      <origin xyz="0 0 0.003" rpy="1.5708 0 0" />
+      <geometry>
+        <mesh filename="package://devotics_arm_description/meshes/visual/Jaula_bolas.stl" scale="0.001 0.001 0.001" />
+      </geometry>
+      <material name="metallic_silver" />
+    </visual>
+    <!-- 3. Central Servo Horn Retainer Plate (Base_04.stl) in the center hole -->
+    <visual>
+      <origin xyz="0 0 0.002" rpy="1.5708 0 0" />
+      <geometry>
+        <mesh filename="package://devotics_arm_description/meshes/visual/Base_04.stl" scale="0.001 0.001 0.001" />
+      </geometry>
+      <material name="devotics_orange" />
+    </visual>
     <collision>
       <origin xyz="0 0 0.006" rpy="0 0 0" />
@@ -57,5 +74,5 @@
       </geometry>
     </collision>
-    <xacro:cylinder_inertia m="0.15" r="0.075" h="0.012" />
+    <xacro:cylinder_inertia m="0.25" r="0.075" h="0.012" />
   </link>
   <!-- ========================================== -->
@@ -70,5 +87,5 @@
     <dynamics damping="0.1" friction="0.1" />
   </joint>
-  <!-- ========================================== -->
+    <!-- ========================================== -->
   <!-- Base Rotation Link (Drum + 2 Side Towers)  -->
   <!-- ========================================== -->
@@ -82,7 +99,7 @@
       <material name="dark_gray" />
     </visual>
-    <!-- Visual 2: Left Tower (aligned with Left shelf) -->
-    <visual>
-      <origin xyz="0 0.0525 0" rpy="1.5708 0 1.5708" />
+    <!-- Visual 2: Left Tower seated on the Left Shelf -->
+    <visual>
+      <origin xyz="0 0.0325 0.035" rpy="1.5708 0 -1.5708" />
       <geometry>
         <mesh filename="package://devotics_arm_description/meshes/visual/Base_03.stl" scale="0.001 0.001 0.001" />
@@ -90,7 +107,7 @@
       <material name="devotics_orange" />
     </visual>
-    <!-- Visual 3: Right Tower (aligned with Right shelf) -->
-    <visual>
-      <origin xyz="0 -0.0525 0" rpy="1.5708 0 -1.5708" />
+    <!-- Visual 3: Right Tower seated on the Right Shelf -->
+    <visual>
+      <origin xyz="0 -0.0325 0.035" rpy="1.5708 0 1.5708" />
       <geometry>
         <mesh filename="package://devotics_arm_description/meshes/visual/Base_03.stl" scale="0.001 0.001 0.001" />
