Commit message: fix: adjust upper arm visual mesh orientation and formatting in URDF xacro

File: devotics_arm_description/urdf/devotics_arm_v1.urdf.xacro (robot description, xacro)
@@ -134,10 +134,10 @@
     <dynamics damping="0.15" friction="0.1" />
   </joint>
-   <!-- ========================================== -->
+  <!-- ========================================== -->
   <!-- Upper Arm Link (185 mm Pivot-to-Pivot)     -->
   <!-- ========================================== -->
   <link name="upper_arm_link">
     <visual>
-      <origin xyz="0 0 0" rpy="1.5708 0 0" />
+      <origin xyz="0 0 0" rpy="1.5708 0 1.5708" />
       <geometry>
         <mesh filename="package://devotics_arm_description/meshes/visual/Brazo_01.stl" scale="0.001 0.001 0.001" />
